Commit message: with contacts; with fixed recording

File: protoverse/data/assets/urdf/g1_29dof_with_sensors.urdf (robot description, URDF)
Before this commit: robot g1_29dof, 138 links, 137 joints
Links:
- removed link left_ankle_roll_link_sensor_20
- removed link left_ankle_roll_link_sensor_21
- removed link left_ankle_roll_link_sensor_22
- removed link left_ankle_roll_link_sensor_23
- removed link left_ankle_roll_link_sensor_24
- removed link left_ankle_roll_link_sensor_25
- removed link left_ankle_roll_link_sensor_26
- removed link left_ankle_roll_link_sensor_27
- removed link left_ankle_roll_link_sensor_28
- removed link left_ankle_roll_link_sensor_29
- removed link left_ankle_roll_link_sensor_30
- removed link left_ankle_roll_link_sensor_31
- removed link left_ankle_roll_link_sensor_32
- removed link left_ankle_roll_link_sensor_33
- removed link left_ankle_roll_link_sensor_34
- removed link left_ankle_roll_link_sensor_35
- removed link left_ankle_roll_link_sensor_36
- removed link left_ankle_roll_link_sensor_37
- removed link left_ankle_roll_link_sensor_38
- removed link left_ankle_roll_link_sensor_39
- removed link left_ankle_roll_link_sensor_40
- removed link left_ankle_roll_link_sensor_41
- removed link left_ankle_roll_link_sensor_42
- removed link left_ankle_roll_link_sensor_43
- removed link left_ankle_roll_link_sensor_44
- removed link left_ankle_roll_link_sensor_45
- removed link left_ankle_roll_link_sensor_46
- removed link left_ankle_roll_link_sensor_47
- removed link left_ankle_roll_link_sensor_48
- removed link right_ankle_roll_link_sensor_20
- removed link right_ankle_roll_link_sensor_21
- removed link right_ankle_roll_link_sensor_22
- removed link right_ankle_roll_link_sensor_23
- removed link right_ankle_roll_link_sensor_24
- removed link right_ankle_roll_link_sensor_25
- removed link right_ankle_roll_link_sensor_26
- removed link right_ankle_roll_link_sensor_27
- removed link right_ankle_roll_link_sensor_28
- removed link right_ankle_roll_link_sensor_29
- removed link right_ankle_roll_link_sensor_30
- removed link right_ankle_roll_link_sensor_31
- removed link right_ankle_roll_link_sensor_32
- removed link right_ankle_roll_link_sensor_33
- removed link right_ankle_roll_link_sensor_34
- removed link right_ankle_roll_link_sensor_35
- removed link right_ankle_roll_link_sensor_36
- removed link right_ankle_roll_link_sensor_37
- removed link right_ankle_roll_link_sensor_38
- removed link right_ankle_roll_link_sensor_39
- removed link right_ankle_roll_link_sensor_40
- removed link right_ankle_roll_link_sensor_41
- removed link right_ankle_roll_link_sensor_42
- removed link right_ankle_roll_link_sensor_43
- removed link right_ankle_roll_link_sensor_44
- removed link right_ankle_roll_link_sensor_45
- removed link right_ankle_roll_link_sensor_46
- removed link right_ankle_roll_link_sensor_47
- removed link right_ankle_roll_link_sensor_48
Joints:
- removed joint left_ankle_roll_link_sensor_20_joint
- removed joint left_ankle_roll_link_sensor_21_joint
- removed joint left_ankle_roll_link_sensor_22_joint
- removed joint left_ankle_roll_link_sensor_23_joint
- removed joint left_ankle_roll_link_sensor_24_joint
- removed joint left_ankle_roll_link_sensor_25_joint
- removed joint left_ankle_roll_link_sensor_26_joint
- removed joint left_ankle_roll_link_sensor_27_joint
- removed joint left_ankle_roll_link_sensor_28_joint
- removed joint left_ankle_roll_link_sensor_29_joint
- removed joint left_ankle_roll_link_sensor_30_joint
- removed joint left_ankle_roll_link_sensor_31_joint
- removed joint left_ankle_roll_link_sensor_32_joint
- removed joint left_ankle_roll_link_sensor_33_joint
- removed joint left_ankle_roll_link_sensor_34_joint
- removed joint left_ankle_roll_link_sensor_35_joint
- removed joint left_ankle_roll_link_sensor_36_joint
- removed joint left_ankle_roll_link_sensor_37_joint
- removed joint left_ankle_roll_link_sensor_38_joint
- removed joint left_ankle_roll_link_sensor_39_joint
- removed joint left_ankle_roll_link_sensor_40_joint
- removed joint left_ankle_roll_link_sensor_41_joint
- removed joint left_ankle_roll_link_sensor_42_joint
- removed joint left_ankle_roll_link_sensor_43_joint
- removed joint left_ankle_roll_link_sensor_44_joint
- removed joint left_ankle_roll_link_sensor_45_joint
- removed joint left_ankle_roll_link_sensor_46_joint
- removed joint left_ankle_roll_link_sensor_47_joint
- removed joint left_ankle_roll_link_sensor_48_joint
- removed joint right_ankle_roll_link_sensor_20_joint
- removed joint right_ankle_roll_link_sensor_21_joint
- removed joint right_ankle_roll_link_sensor_22_joint
- removed joint right_ankle_roll_link_sensor_23_joint
- removed joint right_ankle_roll_link_sensor_24_joint
- removed joint right_ankle_roll_link_sensor_25_joint
- removed joint right_ankle_roll_link_sensor_26_joint
- removed joint right_ankle_roll_link_sensor_27_joint
- removed joint right_ankle_roll_link_sensor_28_joint
- removed joint right_ankle_roll_link_sensor_29_joint
- removed joint right_ankle_roll_link_sensor_30_joint
- removed joint right_ankle_roll_link_sensor_31_joint
- removed joint right_ankle_roll_link_sensor_32_joint
- removed joint right_ankle_roll_link_sensor_33_joint
- removed joint right_ankle_roll_link_sensor_34_joint
- removed joint right_ankle_roll_link_sensor_35_joint
- removed joint right_ankle_roll_link_sensor_36_joint
- removed joint right_ankle_roll_link_sensor_37_joint
- removed joint right_ankle_roll_link_sensor_38_joint
- removed joint right_ankle_roll_link_sensor_39_joint
- removed joint right_ankle_roll_link_sensor_40_joint
- removed joint right_ankle_roll_link_sensor_41_joint
- removed joint right_ankle_roll_link_sensor_42_joint
- removed joint right_ankle_roll_link_sensor_43_joint
- removed joint right_ankle_roll_link_sensor_44_joint
- removed joint right_ankle_roll_link_sensor_45_joint
- removed joint right_ankle_roll_link_sensor_46_joint
- removed joint right_ankle_roll_link_sensor_47_joint
- removed joint right_ankle_roll_link_sensor_48_joint
- joint left_ankle_roll_link_sensor_0_joint: origin xyz=-0.05147892742460647 -0.020779196468829614 -0.035409145057201385 rpy=0 0 0 -> xyz=-0.055637020617723465 -0.01753056049346924 -0.035409145057201385 rpy=0 0 0
- joint left_ankle_roll_link_sensor_10_joint: origin xyz=0.03815935789983044 -0.024326121316740106 -0.035409145057201385 rpy=0 0 0 -> xyz=0.04781141494230334 -0.021126070210746486 -0.035409145057201385 rpy=0 0 0
- joint left_ankle_roll_link_sensor_11_joint: origin xyz=0.07185805629856089 -0.02284244607846517 -0.035409145057201385 rpy=0 0 0 -> xyz=-0.023337149098129915 -0.027376816511906567 -0.035409145057201385 rpy=0 0 0
- joint left_ankle_roll_link_sensor_12_joint: origin xyz=0.10420953773494139 -0.020340784162721975 -0.035409145057201385 rpy=0 0 0 -> xyz=0.1270152921434886 0.026402693238038264 -0.035409145057201385 rpy=0 0 0
- joint left_ankle_roll_link_sensor_13_joint: origin xyz=0.13351999559828798 -0.017105046694074273 -0.035409145057201385 rpy=0 0 0 -> xyz=0.11906076967716217 -0.02979634888470173 -0.035409145057201385 rpy=0 0 0
- joint left_ankle_roll_link_sensor_14_joint: origin xyz=-0.05795339814852556 -0.01035503404033698 -0.035409145057201385 rpy=0 0 0 -> xyz=0.07290523644131497 0.025760665389379885 -0.035409145057201385 rpy=0 0 0
- joint left_ankle_roll_link_sensor_15_joint: origin xyz=-0.026499983852078746 -0.01254755427615068 -0.035409145057201385 rpy=0 0 0 -> xyz=0.024363292923737324 0.010831752146772088 -0.035409145057201385 rpy=0 0 0
- joint left_ankle_roll_link_sensor_16_joint: origin xyz=0.003049850150604592 -0.02444328066435545 -0.035409145057201385 rpy=0 0 0 -> xyz=0.02074342886617637 -0.013454411505767637 -0.035409145057201385 rpy=0 0 0
- joint left_ankle_roll_link_sensor_17_joint: origin xyz=0.040099611243184986 -0.022163588004883588 -0.035409145057201385 rpy=0 0 0 -> xyz=0.113345970228873 0.009750836066674937 -0.035409145057201385 rpy=0 0 0
- joint left_ankle_roll_link_sensor_18_joint: origin xyz=0.07271741908204299 -0.012411505339728467 -0.035409145057201385 rpy=0 0 0 -> xyz=0.07486605616136241 -0.013717407289456382 -0.035409145057201385 rpy=0 0 0
- joint left_ankle_roll_link_sensor_19_joint: origin xyz=0.10457053378734785 -0.011151025291145214 -0.035409145057201385 rpy=0 0 0 -> xyz=0.09925884753465652 -0.03344310075044632 -0.035409145057201385 rpy=0 0 0
- joint left_ankle_roll_link_sensor_1_joint: origin xyz=-0.030403543373492832 -0.027194422708087983 -0.035409145057201385 rpy=0 0 0 -> xyz=0.1408048627815518 -0.00906185914414626 -0.035409145057201385 rpy=0 0 0
- joint left_ankle_roll_link_sensor_2_joint: origin xyz=0.004008545243229822 -0.027817265905054577 -0.035409145057201385 rpy=0 0 0 -> xyz=0.04541489083289126 0.027900194092415006 -0.035409145057201385 rpy=0 0 0
- joint left_ankle_roll_link_sensor_3_joint: origin xyz=0.03728386552887426 -0.02872146074463769 -0.035409145057201385 rpy=0 0 0 -> xyz=0.07325843192029541 -0.03380060481763203 -0.035409145057201385 rpy=0 0 0
- joint left_ankle_roll_link_sensor_4_joint: origin xyz=0.07093099047943345 -0.02619078630258939 -0.035409145057201385 rpy=0 0 0 -> xyz=0.004731578841937134 -0.02784947292223757 -0.035409145057201385 rpy=0 0 0
- joint left_ankle_roll_link_sensor_5_joint: origin xyz=0.10503671665431294 -0.025746526307404365 -0.035409145057201385 rpy=0 0 0 -> xyz=-0.02317839828495936 0.02798237626144621 -0.035409145057201385 rpy=0 0 0
- joint left_ankle_roll_link_sensor_6_joint: origin xyz=0.13085034489631653 -0.023347636684775352 -0.035409145057201385 rpy=0 0 0 -> xyz=0.09899076865652882 0.024958457052427854 -0.035409145057201385 rpy=0 0 0
- joint left_ankle_roll_link_sensor_7_joint: origin xyz=-0.054654310640277905 -0.016594955381014194 -0.035409145057201385 rpy=0 0 0 -> xyz=0.0997927493567405 -0.011936409671415803 -0.035409145057201385 rpy=0 0 0
- joint left_ankle_roll_link_sensor_8_joint: origin xyz=-0.031315424305345486 -0.026428060127047254 -0.035409145057201385 rpy=0 0 0 -> xyz=-0.05797726616714158 0.014480404713548677 -0.035409145057201385 rpy=0 0 0
- joint left_ankle_roll_link_sensor_9_joint: origin xyz=0.0035820337917938823 -0.024652038169573665 -0.035409145057201385 rpy=0 0 0 -> xyz=0.005852564344176935 0.028306550455700824 -0.035409145057201385 rpy=0 0 0
- joint right_ankle_roll_link_sensor_0_joint: origin xyz=-0.05152185988034221 -0.020928998573039936 -0.035409145057201385 rpy=0 0 0 -> xyz=0.0592622877612515 0.03225596051598955 -0.035409145057201385 rpy=0 0 0
- joint right_ankle_roll_link_sensor_10_joint: origin xyz=0.03814782263652075 -0.024497435592205883 -0.035409145057201385 rpy=0 0 0 -> xyz=0.08719900466373262 0.010253541258251989 -0.035409145057201385 rpy=0 0 0
- joint right_ankle_roll_link_sensor_11_joint: origin xyz=0.07187671672392552 -0.022980581989981968 -0.035409145057201385 rpy=0 0 0 -> xyz=0.11918276679729722 -0.029825987792755918 -0.035409145057201385 rpy=0 0 0
- joint right_ankle_roll_link_sensor_12_joint: origin xyz=0.1043953294899373 -0.020356481670025635 -0.035409145057201385 rpy=0 0 0 -> xyz=0.047853862920995485 -0.021288241919016404 -0.035409145057201385 rpy=0 0 0
- joint right_ankle_roll_link_sensor_13_joint: origin xyz=0.1333885536811086 -0.01707114036162157 -0.035409145057201385 rpy=0 0 0 -> xyz=0.13669402246317006 0.01762913770410026 -0.035409145057201385 rpy=0 0 0
- joint right_ankle_roll_link_sensor_14_joint: origin xyz=-0.05794387204414322 -0.010486026496501518 -0.035409145057201385 rpy=0 0 0 -> xyz=0.08706002214229262 0.0342641778290631 -0.035409145057201385 rpy=0 0 0
- joint right_ankle_roll_link_sensor_15_joint: origin xyz=-0.026499991257030585 -0.012646673083963802 -0.035409145057201385 rpy=0 0 0 -> xyz=-0.046314858565519076 -0.025671661221727718 -0.035409145057201385 rpy=0 0 0
- joint right_ankle_roll_link_sensor_16_joint: origin xyz=0.0030461061646167033 -0.024635589597541026 -0.035409145057201385 rpy=0 0 0 -> xyz=0.11331249280105574 0.009674593082315731 -0.035409145057201385 rpy=0 0 0
- joint right_ankle_roll_link_sensor_17_joint: origin xyz=0.0396506008242065 -0.02266048856743494 -0.035409145057201385 rpy=0 0 0 -> xyz=-0.026499986090228213 0.010744321969178997 -0.035409145057201385 rpy=0 0 0
- joint right_ankle_roll_link_sensor_18_joint: origin xyz=0.0727271252849399 -0.0124747704520709 -0.035409145057201385 rpy=0 0 0 -> xyz=0.032736116758765976 0.030724363625874825 -0.035409145057201385 rpy=0 0 0
- joint right_ankle_roll_link_sensor_19_joint: origin xyz=0.10457482796474882 -0.011233994821511363 -0.035409145057201385 rpy=0 0 0 -> xyz=0.0625661186581081 0.01184758864172776 -0.035409145057201385 rpy=0 0 0
- joint right_ankle_roll_link_sensor_1_joint: origin xyz=-0.03041028205981262 -0.02738614059429512 -0.035409145057201385 rpy=0 0 0 -> xyz=-0.06105424633451832 -0.007378061747620619 -0.035409145057201385 rpy=0 0 0
- joint right_ankle_roll_link_sensor_2_joint: origin xyz=0.004059180358040036 -0.028005031016869932 -0.035409145057201385 rpy=0 0 0 -> xyz=0.14080649614334106 -0.009282348677515984 -0.035409145057201385 rpy=0 0 0
- joint right_ankle_roll_link_sensor_3_joint: origin xyz=0.03744334661330561 -0.02886953889508301 -0.035409145057201385 rpy=0 0 0 -> xyz=0.02097146717677151 -0.029712819657697946 -0.035409145057201385 rpy=0 0 0
- joint right_ankle_roll_link_sensor_4_joint: origin xyz=0.07091681886267169 -0.026382393274782357 -0.035409145057201385 rpy=0 0 0 -> xyz=-0.009652182537602937 0.02755135291814013 -0.035409145057201385 rpy=0 0 0
- joint right_ankle_roll_link_sensor_5_joint: origin xyz=0.10471389989576807 -0.025953373021419368 -0.035409145057201385 rpy=0 0 0 -> xyz=0.08573751036989502 -0.02626644118289932 -0.035409145057201385 rpy=0 0 0
- joint right_ankle_roll_link_sensor_6_joint: origin xyz=0.13094720244407654 -0.023374522104859352 -0.035409145057201385 rpy=0 0 0 -> xyz=0.11035671830177307 0.03188828378915787 -0.035409145057201385 rpy=0 0 0
- joint right_ankle_roll_link_sensor_7_joint: origin xyz=-0.05468999799628186 -0.01672481232289301 -0.035409145057201385 rpy=0 0 0 -> xyz=-0.023341336837108352 -0.027571243090429517 -0.035409145057201385 rpy=0 0 0
- joint right_ankle_roll_link_sensor_8_joint: origin xyz=-0.0313277469941269 -0.026617733549849767 -0.035409145057201385 rpy=0 0 0 -> xyz=0.02438298362611916 0.010755967509670474 -0.035409145057201385 rpy=0 0 0
- joint right_ankle_roll_link_sensor_9_joint: origin xyz=0.00357793349989041 -0.024846397227688177 -0.035409145057201385 rpy=0 0 0 -> xyz=-0.04199344780509925 0.026611821000404094 -0.035409145057201385 rpy=0 0 0
